Commit message: ldlidar added

File: urdf/roboclaw_description.urdf.xacro (robot description, xacro)
@@ -260,4 +260,28 @@
     </link>
       <!-- end -->
+      <!-- start ldlarar -->
+    <joint name="base_ldlidar_joint" type="fixed">
+      <parent link="base_link"/>
+      <child link="ldlidar_base"/>
+      <origin xyz="0.4 0 0.8" rpy="0 0.18 0"/>
+    </joint>
+    <link name="ldlidar_base">
+        <visual>
+            <origin xyz="0 0 0" rpy="0 0 0"/>
+            <geometry>
+                <mesh filename="package://ldlidar_node/urdf/model/LD19.stl" scale="0.001 0.001 0.001" />
+            </geometry>
+            <material name="ldlidar_mat">
+                <color rgba="0.8 0.8 0.8 0.8"/>
+            </material>
+        </visual>
+    </link>
+    <joint name="ldlidar_link_joint" type="fixed">
+        <parent link="ldlidar_base"/>
+        <child link="ldlidar_link"/>
+        <origin xyz="0 0 0.02745" rpy="0 0 0" />
+    </joint>
+    <link name="ldlidar_link" />
+      <!-- end ldladar -->
   </xacro:macro>
 </robot>

Commit message: oriented lllidar, kinda

File: urdf/roboclaw_description.urdf.xacro (robot description, xacro)
@@ -264,15 +264,16 @@
       <parent link="base_link"/>
       <child link="ldlidar_base"/>
-      <origin xyz="0.4 0 0.8" rpy="0 0.18 0"/>
+      <origin xyz="0.0 0 0.4" rpy="0 0.0 0"/>
     </joint>
     <link name="ldlidar_base">
         <visual>
-            <origin xyz="0 0 0" rpy="0 0 0"/>
-            <geometry>
-                <mesh filename="package://ldlidar_node/urdf/model/LD19.stl" scale="0.001 0.001 0.001" />
-            </geometry>
-            <material name="ldlidar_mat">
-                <color rgba="0.8 0.8 0.8 0.8"/>
-            </material>
+         <origin xyz="0.0 0.0 0.0" rpy="0.0 0.0 0.0"/>
+              <geometry>
+                  <cylinder radius="0.1" length="0.1"/>
+              </geometry>
+              <material name="green">
+                  <!-- <color rgba="1.0 0.0 1.0 1.0"/> -->
+                  <texture filename=""/>
+              </material>
         </visual>
     </link>

Commit message: fixed lidar mount

File: urdf/roboclaw_description.urdf.xacro (robot description, xacro)
@@ -264,5 +264,5 @@
       <parent link="base_link"/>
       <child link="ldlidar_base"/>
-      <origin xyz="0.0 0 0.4" rpy="0 0.0 0"/>
+      <origin xyz="0.0 0 0.5" rpy="0 0.0 ${PI}"/>
     </joint>
     <link name="ldlidar_base">
