Commit message: fixed lidar mount

File: install/ag_sml_bringup/share/ag_sml_bringup/urdf/roboclaw_description.urdf.xacro (robot description, xacro)
@@ -183,5 +183,5 @@
           </visual>
       </link>
-  <!-- *********************** GPS SETUP  **********************************  -->
+  <!-- *********************** GPS SETUP **********************************  -->
     <joint name="gps_joint" type="fixed">
       <parent link="base_link"/>
@@ -264,5 +264,5 @@
       <parent link="base_link"/>
       <child link="ldlidar_base"/>
-      <origin xyz="0.0 0 0.5" rpy="0 0.0 ${PI}"/>
+      <origin xyz="0.0 0 0.5" rpy="0 0.0 ${pi}"/>
     </joint>
     <link name="ldlidar_base">

Commit message: changed velocity

File: install/ag_sml_bringup/share/ag_sml_bringup/urdf/roboclaw_description.urdf.xacro (robot description, xacro)
@@ -183,5 +183,5 @@
           </visual>
       </link>
-  <!-- *********************** GPS SETUP **********************************  -->
+  <!-- *********************** GPS SETUP  **********************************  -->
     <joint name="gps_joint" type="fixed">
       <parent link="base_link"/>
@@ -264,5 +264,5 @@
       <parent link="base_link"/>
       <child link="ldlidar_base"/>
-      <origin xyz="0.0 0 0.5" rpy="0 0.0 ${pi}"/>
+      <origin xyz="0.0 0 0.5" rpy="0 0.0 ${PI}"/>
     </joint>
     <link name="ldlidar_base">
